Commit message: trajopt integration completed, ik and trajectory optimization work

File: models/hsrb_whole_body.urdf (robot description, URDF)
Before this commit: robot hsrb, 47 links, 46 joints
Joints:
- joint base_t_joint: limit lower=-10.0 upper=10.0 effort=300.0 velocity=0.2 -> lower=-3.14 upper=3.14 effort=300.0 velocity=2.5
